File: X15-DataConversion.sch (EAGLE design)
At the start: 22 parts

Commit message: used the wrong connector so fixed that
Parts:
- U$1: value DATACONV->BACKPLANE -> BACKPLANE->DATACONV; device X15-Data-Conversion-Parts:DATACONV->BACKPLANE -> X15-Data-Conversion-Parts:BACKPLANE->DATACONV
Changed lines of the file:
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@@
 <part name="GND6" library="supply1" library_urn="urn:adsk.eagle:library:371" deviceset="GND" device=""/>
 <part name="CONNECTOR1" library="X15-Data-Conversion-Parts" deviceset="SWD_CONN" device="" package3d_urn="urn:adsk.eagle:package:38192072/1" value="3V3 -SWCLK-GND-SWDIO- NRST"/>
-<part name="U$1" library="X15-Data-Conversion-Parts" deviceset="DATACONV-&gt;BACKPLANE" device="" package3d_urn="urn:adsk.eagle:package:38192071/2"/>
+<part name="U$1" library="X15-Data-Conversion-Parts" deviceset="BACKPLANE-&gt;DATACONV" device="" package3d_urn="urn:adsk.eagle:package:38192070/1"/>
 <part name="CAN_TRANCEIVER" library="X15-Data-Conversion-Parts" deviceset="MAX3058ASA+" device="" package3d_urn="urn:adsk.eagle:package:38192068/2"/>
 <part name="C6" library="SparkFun-RF" deviceset="0.1UF" device="-0603-25V-5%" value="0.1uF"/>
